Commit message: fixed camera orientation problem; fixed scale problem, update duckietown_udem.world environment.

File: src/duckiebot_description/urdf/duckiebot.xacro (robot description, xacro)
@@ -144,5 +144,5 @@
     <pose>0 0 0 0 0 0</pose>
     <collision>
-      <origin xyz="0 -0.2 -0.7" rpy="0 0 0"/>
+      <origin xyz="-0.05 0 -0.055" rpy="0 -0.1 0"/>
       <geometry>
         <mesh filename="package://duckiebot_description/meshes/duckiebot_camera.dae"/>
@@ -150,5 +150,5 @@
     </collision>
     <visual name='camvisual'>
-      <origin xyz="0 -0.2 -0.7" rpy=" 0 0 0"/>
+      <origin xyz="-0.05 0 -0.055" rpy=" 0 -0.1 0"/>
       <geometry>
         <mesh filename="package://duckiebot_description/meshes/duckiebot_camera.dae"/>
@@ -162,7 +162,8 @@
     </inertial>
   </link>
+<!-- This joint info decides the pos of camera. Pitch(p in rpy) is angle to control orientation for duckiebot camera.After change values here, you need to change the pos info in collision part anf visual part just above.-->
   <joint name="camera_joint" type="fixed">
     <axis xyz="0 0 0" />
-    <origin xyz="0 0.2 0.7" rpy="0 0 0"/>
+    <origin xyz="0.05 0 0.05" rpy="0 0.1 0"/>
     <parent link="chassis"/>
     <child link="camera"/>
